Commit message: Corrige orientacao de montagem do Ouster: azimute zero do sensor estava 90 graus errado em relacao a frente do robo. Confirmado visualmente pelo usuario e ajustado via ouster_yaw=-90deg no joint os_sensor_joint.
Co-Authored-By: Claude Sonnet 5 <noreply@anthropic.com>

File: ros2_ws/src/mobi_description/urdf/mobi.urdf.xacro (robot description, xacro)
@@ -50,4 +50,9 @@
   <xacro:property name="mast_length" value="0.55"/>
   <xacro:property name="mast_radius" value="0.006"/>
+  <!-- O "azimute zero" do Ouster (referencia fisica do sensor, geralmente
+       perto do conector) nao sai alinhado com a frente do robo so por causa
+       de como ele foi montado na caixa. Ajuste este valor se a orientacao
+       mudar num remonte futuro. -->
+  <xacro:property name="ouster_yaw" value="${-pi/2}"/>
   <!-- materiais (so visual) -->
   <material name="mobi_body_gray">
@@ -126,5 +131,5 @@
     <parent link="base_link"/>
     <child link="os_sensor"/>
-    <origin xyz="${ouster_x} 0 ${base_height + ouster_standoff}" rpy="0 0 0"/>
+    <origin xyz="${ouster_x} 0 ${base_height + ouster_standoff}" rpy="0 0 ${ouster_yaw}"/>
   </joint>
   <!-- D435i + T265 (face frontal) -->

Commit message: Corrige montagem do Ouster com o driver jazzy-0.14.2: yaw +90, x 0.20 m, caixa 0.32 m.
Medido com o robo parado: chao a +8 cm de base_link (base_height era 0.40),
tampo do robo visivel so atras do sensor (Ouster ~15 cm da borda frontal) e
frente = lado do Ouster (confirmado pelo usuario). O -90 validado antes era do
driver Humble; as versoes diferem em 180 graus no frame do sensor.
Margem traseira do filtro de corpo e da pegada do Nav2 ampliada para -0.40 m.

Co-Authored-By: Claude Opus 5.5 <noreply@anthropic.com>

File: ros2_ws/src/mobi_description/urdf/mobi.urdf.xacro (robot description, xacro)
@@ -32,5 +32,7 @@
   <xacro:property name="base_length" value="0.70"/>
   <xacro:property name="base_width"  value="0.50"/>
-  <xacro:property name="base_height" value="0.40"/>
+  <!-- 0.32 medido: com 0.40 o chao aparecia a +8 cm de base_link na nuvem do
+       Ouster (ajuste de plano no chao, robo parado, 2026-10-06). -->
+  <xacro:property name="base_height" value="0.32"/>
   <xacro:property name="wheel_radius" value="0.05"/>
   <xacro:property name="wheel_width"  value="0.03"/>
@@ -38,5 +40,7 @@
   <xacro:property name="wheel_inset_y" value="0.03"/>
   <xacro:property name="tof_size" value="0.02"/>
-  <xacro:property name="ouster_x" value="${base_length/2 - 0.10}"/>
+  <!-- Medido pelo tampo visto do sensor: a borda frontal fica ~15 cm a frente
+       do Ouster e o tampo se estende ~0.6 m para tras. -->
+  <xacro:property name="ouster_x" value="${base_length/2 - 0.15}"/>
   <xacro:property name="ouster_radius" value="0.045"/>
   <xacro:property name="ouster_height" value="0.07"/>
@@ -53,6 +57,10 @@
        perto do conector) nao sai alinhado com a frente do robo so por causa
        de como ele foi montado na caixa. Ajuste este valor se a orientacao
-       mudar num remonte futuro. -->
-  <xacro:property name="ouster_yaw" value="${-pi/2}"/>
+       mudar num remonte futuro.
+       +90 graus com o driver ouster-ros jazzy-0.14.2 (frente do robo = lado
+       do Ouster, confirmado pelo usuario). Com o driver Humble antigo o valor
+       validado era -90: as versoes diferem em 180 graus no frame do sensor.
+       Conferir com ./mobi.sh check-yaw sempre que trocar o driver. -->
+  <xacro:property name="ouster_yaw" value="${pi/2}"/>
   <!-- materiais (so visual) -->
   <material name="mobi_body_gray">

Commit message: Ouster yaw 0 (ajuste visual do usuario); Nav2 e localizacao funcionando na Thor.
- URDF: ouster_yaw 0 (corpo girado 90 graus anti-horario em torno da frente).
- slam.launch: localizacao parte da origem do mapa (RGBD/StartAtOrigin) e
  aceita a 1a localizacao (RGBD/MaxOdomCacheSize 0); so com LiDAR o rtabmap
  nao relocaliza do nada e nao publicava o mapa com o robo parado.
- slam_icp: remove scan_downsampling_step (icp_odometry abortava no kdtree
  do PCL com a nuvem organizada do Ouster).
- nav2: collision_monitor sem base_shift_correction (odometria ICP atrasada
  fazia o monitor zerar todo comando) e transform_tolerance 0.5.
- compose: PYTHONUNBUFFERED nos servicos ROS 1 (logs do mux em tempo real).

Co-Authored-By: Claude Opus 5.5 <noreply@anthropic.com>

File: ros2_ws/src/mobi_description/urdf/mobi.urdf.xacro (robot description, xacro)
@@ -58,9 +58,10 @@
        de como ele foi montado na caixa. Ajuste este valor se a orientacao
        mudar num remonte futuro.
-       +90 graus com o driver ouster-ros jazzy-0.14.2 (frente do robo = lado
-       do Ouster, confirmado pelo usuario). Com o driver Humble antigo o valor
-       validado era -90: as versoes diferem em 180 graus no frame do sensor.
+       0 grau com o driver ouster-ros jazzy-0.14.2: ajustado pelo usuario
+       comparando o corpo do robo com a nuvem no RViz (corpo girado 90 graus
+       anti-horario em torno da frente, onde fica o Ouster). Com o driver
+       Humble antigo o valor validado era -90.
        Conferir com ./mobi.sh check-yaw sempre que trocar o driver. -->
-  <xacro:property name="ouster_yaw" value="${pi/2}"/>
+  <xacro:property name="ouster_yaw" value="0"/>
   <!-- materiais (so visual) -->
   <material name="mobi_body_gray">
